Commit message: implemented human interface + added Hokuyo laser to robot mode + example of TF listener (ros tutorials) + modified launch files

File: urdf/robot.xacro (robot description, xacro)
@@ -2,6 +2,10 @@
 <robot name="robot" xmlns:xacro="http://www.ros.org/wiki/xacro">
   <!-- materials -->
- <xacro:include filename="$(find exp_assignment2)/urdf/materials.xacro" />
- <xacro:include filename="$(find exp_assignment2)/urdf/robot.gazebo" />
+ <xacro:include filename="$(find exp_assignment3)/urdf/materials.xacro" />
+ <xacro:include filename="$(find exp_assignment3)/urdf/robot.gazebo" />
+ <xacro:property name="chassis_length" value="0.5" />
+ <xacro:property name="chassis_width" value="0.3" />
+ <xacro:property name="chassis_height" value="0.07" />
+ <xacro:property name="chassis_mass" value="6" />
  <xacro:property name="length_wheel" value="0.04" />
  <xacro:property name="radius_wheel" value="0.10" />
@@ -20,38 +24,4 @@
                 iyy="${mass*(w*w+d*d)/12}" iyz = "0" izz="${mass*(w*w+h*h)/12}" />
  </xacro:macro>
- <!-- <xacro:macro name="link_ear" params="name">
-   <link name="${name}">
-            <inertial>
-              <mass value="0.1"/>
-              <origin rpy="0 0 0" xyz="0 0 0"/>
-              <inertia ixx="0.000526666666667" ixy="0" ixz="0" iyy="0.000526666666667" iyz="0" izz="0.001"/>
-	      <xacro:box_inertia mass="0.1" w="0.05" h="0.03" d="0.034"/>
-            </inertial>
-            <collision name="${name}_collision">
-              <origin rpy="0 0 1.5708" xyz="0 0 0"/>
-              <geometry>
-                <box size="0.034 0.05 0.03"/>
-              </geometry>
-            </collision>
-            <visual name="${name}_visual">
-              <origin rpy="0 0 0" xyz="0 0 0"/>
-              <geometry>
-                <box size="0.034 0.05 0.03"/>
-              </geometry>
-		<material name="blue" />
-            </visual>
-        </link>
- </xacro:macro>
-    <xacro:macro name="joint_ear" params="name child origin_xyz">
-      <joint name="${name}" type="fixed">
-        <origin rpy="0 0 0" xyz="${origin_xyz}"/>
-        <child link="${child}"/>
-        <parent link="head_link"/>
-        <axis rpy="0 0 0" xyz="0 0 1"/>
-        <limit effort="10000" velocity="1000"/>
-        <joint_properties damping="1.0" friction="1.0"/>
-      </joint>
-    </xacro:macro>
--->
     <xacro:macro name="link_wheel" params="name">
         <link name="${name}">
@@ -225,5 +195,5 @@
   <xacro:joint_ear name="joint_right_ear"  child="link_right_ear"  origin_xyz="0 0.08 0.08"  />
   <xacro:joint_ear name="joint_left_ear"   child="link_left_ear"   origin_xyz="0 -0.08 0.08"  /> -->
-<!-- transmission -->
+<!-- transmission
 <transmission name="head_joint_trans">
 	<type>transmission_interface/SimpleTransmission</type>
@@ -235,4 +205,32 @@
 		<mechanicalInterface>1</mechanicalInterface>
 	</actuator>
-</transmission>
+</transmission> -->
+<link name="hokuyo_link">
+	    <collision>
+	      <origin xyz="0 0 0.00125" rpy="0 0 0"/>
+	      <geometry>
+		<box size="0.025 0.025 0.025"/>
+	      </geometry>
+	    </collision>
+	    <visual>
+	      <origin xyz="0 0 0.0125" rpy="0 0 0"/>
+	      <geometry>
+		<box size="0.025 0.025 0.025"/>
+	      </geometry>
+	      <material name="red">
+		<color rgba="1 0 0 1"/>
+	      </material>
+	    </visual>
+	    <inertial>
+	      <mass value="1e-5" />
+	      <origin xyz="0 0 0" rpy="0 0 0"/>
+	      <inertia ixx="1e-6" ixy="0" ixz="0" iyy="1e-6" iyz="0" izz="1e-6" />
+	    </inertial>
+  </link>
+  <joint name="hokuyo_joint" type="fixed">
+	    <axis xyz="0 1 0" />
+	    <origin xyz="0.27 0 0.025" rpy="0 0 0"/>
+	    <parent link="base_link"/>
+	    <child link="hokuyo_link"/>
+	 </joint>
 </robot>

Commit message: fix some bugs

File: urdf/robot.xacro (robot description, xacro)
@@ -50,5 +50,5 @@
         <origin rpy="0 0 0" xyz="${origin_xyz}"/>
         <child link="${child}"/>
-        <parent link="base_link"/>
+        <parent link="link_chassis"/>
         <axis rpy="0 0 0" xyz="0 1 0"/>
         <limit effort="10000" velocity="1000"/>
@@ -57,5 +57,5 @@
     </xacro:macro>
 <!-- _______________base link____________________  -->
-  <link name="base_link">
+  <link name="link_chassis">
     <!-- pose and inertial -->
     <pose>0 0 0.1 0 0 0</pose>
@@ -132,5 +132,5 @@
   	<limit effort="1000.0" lower="-3.14" upper="3.14" velocity="0.2"/>
   	<origin rpy="0 0 0" xyz="0.15 0 0.035"/> <!-- half the height of the base link -->
-  	<parent link="base_link"/>
+  	<parent link="link_chassis"/>
   	<child link="neck_link"/>
   </joint>
@@ -190,20 +190,4 @@
     <child link="camera_link"/>
   </joint>
-<!-- hears definition -->
-  <!-- <xacro:link_ear name="link_right_ear" />
-  <xacro:link_ear name="link_left_ear" />
-  <xacro:joint_ear name="joint_right_ear"  child="link_right_ear"  origin_xyz="0 0.08 0.08"  />
-  <xacro:joint_ear name="joint_left_ear"   child="link_left_ear"   origin_xyz="0 -0.08 0.08"  /> -->
-<!-- transmission
-<transmission name="head_joint_trans">
-	<type>transmission_interface/SimpleTransmission</type>
-	<joint name="head_joint">
-		<hardwareInterface>hardware_interface/EffortJointInterface</hardwareInterface>
-	</joint>
-	<actuator name="motor1">
-		<hardwareInterface>hardware_interface/EffortJointInterface</hardwareInterface>
-		<mechanicalInterface>1</mechanicalInterface>
-	</actuator>
-</transmission> -->
 <link name="hokuyo_link">
 	    <collision>
@@ -231,5 +215,5 @@
 	    <axis xyz="0 1 0" />
 	    <origin xyz="0.27 0 0.025" rpy="0 0 0"/>
-	    <parent link="base_link"/>
+	    <parent link="link_chassis"/>
 	    <child link="hokuyo_link"/>
 	 </joint>

Commit message: FIXED SWITCH BETWEEN FIND AND PLAY, ADJUST ROBOT MODEL, TUNED CORRECTLY THE TRACKING

File: urdf/robot.xacro (robot description, xacro)
@@ -109,8 +109,8 @@
   <link name="neck_link">
   	<inertial>
-  		<mass value="0.025"/>
+  		<mass value="0.3"/>
   		<origin xyz="0 0 0" rpy="0 0 0" />
-  		<!--<inertia ixx="0.000010279" ixy="0" ixz="0" iyy="0.000010279" iyz="0" izz="0.000007225"/>-->
-		<xacro:cylinder_inertia mass="0.2" r="${neck_radius}" l="${neck_length}" />
+  		<!--<inertia ixx="0.0" ixy="0" ixz="0" iyy="0.0" iyz="0" izz="0.0"/>-->
+		<xacro:cylinder_inertia mass="0.0" r="${neck_radius}" l="${neck_length}" />
   	</inertial>
   	<collision>
@@ -156,5 +156,5 @@
   	</visual>
 </link>
-  <joint name="head_joint" type="revolute">
+  <joint name="head_joint" type="fixed">
   	<axis xyz="0 0 1"/>
   	<limit effort="1000.0" lower="-1.8" upper="1.8" velocity="0.5"/>
